File: standalone/kicad/arduino_standalone/arduino_standalone.kicad_sch (KiCad schematic)
At the start: 9 parts, among them J1 Bateria, U1 L7805CV

Commit message: Início do esquemático do ATmega328P
Parts:
- added D3: 1N4148, symbol Device:D
- added R2: 10K, symbol Device:R
- added SW1: Botão, symbol Switch:SW_Push
- added U2: ATMEGA328P-PU, Cofre_Celular:28P3_ATM, symbol Computacao_Raiz:ATMEGA328P-PU
Connections:
- net +5V: now also D3.1 (K), R2.1
- net GND: now also SW1.1, U2.22 (GND), U2.8 (GND)
- new net AREF: U2.21 (AREF)
- new net AVCC: U2.20 (AVCC)
- new net RESET: D3.2 (A), R2.2, SW1.2, U2.1 (PC6)
- new net VCC: U2.7 (VCC)
- new net XTAL1: U2.9 (PB6)
- new net XTAL2: U2.10 (PB7)
- no-connect marks 0 -> 20
Other:
- note added: "Circuito de reset"
- note added: "Microcontrolador ATmega328P-PU"
- note added: "Tensões de referência"
- note removed: "Tensões de Referência"

Commit message: Finalização versão em português
Parts:
- added C5, C6: 22pF, symbol Device:C
- added C7, C8, C9: 100nF, symbol Device:C
- added L1: 10uH, symbol Device:L
- added R3: 1M, symbol Device:R
- added X1: 16MHz, PCM_Crystal_AKL:Crystal_HC18-U_Vertical, symbol PCM_Crystal_AKL:HC18_Vertical
- U2: footprint Cofre_Celular:28P3_ATM -> Computacao_Raiz:28P3_ATM
Connections:
- net AVCC is gone; now on net +5V: U2.20 (AVCC)
- net VCC is gone; now on net +5V: U2.7 (VCC)
- net +5V: now also C7.2, C8.2, L1.1, L1.2
- net GND: now also C5.2, C6.2, C7.1, C8.1, C9.2
- net XTAL1: now also C6.1, R3.1, X1.1
- net XTAL2: now also C5.1, R3.2, X1.2
- net AREF: no longer names the net of U2.21 (AREF)
- net AREF: now also C9.1
Other:
- note added: "Clock externo"
- moved on the sheet: U2
